File: Design/SCRController/SCRController.kicad_sch (KiCad schematic)
At the start: 24 parts, among them Q1 2N2907A, Q2 2N2222A, Q3 2N2222A, Q4 2N2907A, U1 TL084, U2 TL084

Commit message: Se agregaron footprints basicas, pero falta etapa 1 y 5
Parts:
- C1, C3: footprint PCM_Capacitor_THT_AKL:C_Disc_D3.0mm_W1.6mm_P2.50mm -> Capacitor_THT:CP_Radial_D8.0mm_P3.80mm
- D3, D4, D5, D6: footprint PCM_Diode_THT_AKL:D_DO-35_SOD27_P7.62mm_Horizontal -> Diode_THT:D_5W_P12.70mm_Horizontal
- Q1, Q2, Q3, Q4: footprint PCM_Package_TO_SOT_THT_AKL:TO-18-3_EBC -> Package_TO_SOT_THT:TO-92_HandSolder
- R10, R12, R13, R14, R15, R16, R17, R18, R19, R3, R4, R9: footprint (none) -> Resistor_THT:R_Axial_DIN0411_L9.9mm_D3.6mm_P15.24mm_Horizontal
- U1, U2: footprint (none) -> Package_DIP:CERDIP-14_W7.62mm_SideBrazed
Changed lines of the file:
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@@
 			)
 		)
-		(property "Footprint" "PCM_Package_TO_SOT_THT_AKL:TO-18-3_EBC"
+		(property "Footprint" "Package_TO_SOT_THT:TO-92_HandSolder"
 			(at 82.55 66.04 0)
 			(effects
@@
 			)
 		)
-		(property "Footprint" ""
+		(property "Footprint" "Resistor_THT:R_Axial_DIN0411_L9.9mm_D3.6mm_P15.24mm_Horizontal"
 			(at 104.902 100.33 90)
 			(effects
@@
 			)
 		)
-		(property "Footprint" ""
+		(property "Footprint" "Resistor_THT:R_Axial_DIN0411_L9.9mm_D3.6mm_P15.24mm_Horizontal"
 			(at 79.502 125.73 90)
 			(effects
@@
 			)
 		)
-		(property "Footprint" ""
+		(property "Footprint" "Resistor_THT:R_Axial_DIN0411_L9.9mm_D3.6mm_P15.24mm_Horizontal"
 			(at 103.632 29.21 90)
 			(effects
@@
 			)
 		)
-		(property "Footprint" ""
+		(property "Footprint" "Resistor_THT:R_Axial_DIN0411_L9.9mm_D3.6mm_P15.24mm_Horizontal"
 			(at 66.04 70.358 90)
 			(effects
@@
 			)
 		)
-		(property "Footprint" ""
+		(property "Footprint" "Resistor_THT:R_Axial_DIN0411_L9.9mm_D3.6mm_P15.24mm_Horizontal"
 			(at 67.31 141.478 90)
 			(effects
@@
 			)
 		)
-		(property "Footprint" ""
+		(property "Footprint" "Resistor_THT:R_Axial_DIN0411_L9.9mm_D3.6mm_P15.24mm_Horizontal"
 			(at 103.632 49.53 90)
 			(effects
@@
 			)
 		)
-		(property "Footprint" "PCM_Diode_THT_AKL:D_DO-35_SOD27_P7.62mm_Horizontal"
+		(property "Footprint" "Diode_THT:D_5W_P12.70mm_Horizontal"
 			(at 135.89 132.08 0)
 			(effects
@@
 			)
 		)
-		(property "Footprint" "PCM_Capacitor_THT_AKL:C_Disc_D3.0mm_W1.6mm_P2.50mm"
+		(property "Footprint" "Capacitor_THT:CP_Radial_D8.0mm_P3.80mm"
 			(at 91.1352 127 0)
 			(effects
@@
 			)
 		)
-		(property "Footprint" ""
+		(property "Footprint" "Package_DIP:CERDIP-14_W7.62mm_SideBrazed"
 			(at 41.91 22.86 0)
 			(effects
@@
 			)
 		)
-		(property "Footprint" "PCM_Diode_THT_AKL:D_DO-35_SOD27_P7.62mm_Horizontal"
+		(property "Footprint" "Diode_THT:D_5W_P12.70mm_Horizontal"
 			(at 135.89 64.77 0)
 			(effects
@@
 			)
 		)
-		(property "Footprint" ""
+		(property "Footprint" "Package_DIP:CERDIP-14_W7.62mm_SideBrazed"
 			(at 43.18 137.16 0)
 			(effects
@@
 			)
 		)
-		(property "Footprint" "PCM_Package_TO_SOT_THT_AKL:TO-18-3_EBC"
+		(property "Footprint" "Package_TO_SOT_THT:TO-92_HandSolder"
 			(at 83.82 137.16 0)
 			(effects
@@
 			)
 		)
-		(property "Footprint" ""
+		(property "Footprint" "Package_DIP:CERDIP-14_W7.62mm_SideBrazed"
 			(at 123.19 62.23 0)
 			(effects
@@
 			)
 		)
-		(property "Footprint" "PCM_Diode_THT_AKL:D_DO-35_SOD27_P7.62mm_Horizontal"
+		(property "Footprint" "Diode_THT:D_5W_P12.70mm_Horizontal"
 			(at 58.42 68.58 0)
 			(effects
@@
 			)
 		)
-		(property "Footprint" ""
+		(property "Footprint" "Resistor_THT:R_Axial_DIN0411_L9.9mm_D3.6mm_P15.24mm_Horizontal"
 			(at 143.002 139.7 90)
 			(effects
@@
 			)
 		)
-		(property "Footprint" ""
+		(property "Footprint" "Package_DIP:CERDIP-14_W7.62mm_SideBrazed"
 			(at 43.18 66.04 0)
 			(effects
@@
 			)
 		)
-		(property "Footprint" ""
+		(property "Footprint" "Package_DIP:CERDIP-14_W7.62mm_SideBrazed"
 			(at 123.19 129.54 0)
 			(effects
@@
 			)
 		)
-		(property "Footprint" "PCM_Capacitor_THT_AKL:C_Disc_D3.0mm_W1.6mm_P2.50mm"
+		(property "Footprint" "Capacitor_THT:CP_Radial_D8.0mm_P3.80mm"
 			(at 89.8652 55.88 0)
 			(effects
@@
 			)
 		)
-		(property "Footprint" ""
+		(property "Footprint" "Resistor_THT:R_Axial_DIN0411_L9.9mm_D3.6mm_P15.24mm_Horizontal"
 			(at 87.122 27.94 90)
 			(effects
@@
 			)
 		)
-		(property "Footprint" ""
+		(property "Footprint" "Resistor_THT:R_Axial_DIN0411_L9.9mm_D3.6mm_P15.24mm_Horizontal"
 			(at 104.902 120.65 90)
 			(effects
@@
 			)
 		)
-		(property "Footprint" ""
+		(property "Footprint" "Resistor_THT:R_Axial_DIN0411_L9.9mm_D3.6mm_P15.24mm_Horizontal"
 			(at 143.002 72.39 90)
 			(effects
@@
 			)
 		)
-		(property "Footprint" ""
+		(property "Footprint" "Resistor_THT:R_Axial_DIN0411_L9.9mm_D3.6mm_P15.24mm_Horizontal"
 			(at 78.232 54.61 90)
 			(effects
@@
 			)
 		)
-		(property "Footprint" "PCM_Package_TO_SOT_THT_AKL:TO-18-3_EBC"
+		(property "Footprint" "Package_TO_SOT_THT:TO-92_HandSolder"
 			(at 87.63 105.41 0)
 			(effects
@@
 			)
 		)
-		(property "Footprint" ""
+		(property "Footprint" "Resistor_THT:R_Axial_DIN0411_L9.9mm_D3.6mm_P15.24mm_Horizontal"
 			(at 88.392 99.06 90)
 			(effects
@@
 			)
 		)
-		(property "Footprint" "PCM_Diode_THT_AKL:D_DO-35_SOD27_P7.62mm_Horizontal"
+		(property "Footprint" "Diode_THT:D_5W_P12.70mm_Horizontal"
 			(at 59.69 139.7 0)
 			(effects
@@
 			)
 		)
-		(property "Footprint" "PCM_Package_TO_SOT_THT_AKL:TO-18-3_EBC"
+		(property "Footprint" "Package_TO_SOT_THT:TO-92_HandSolder"
 			(at 86.36 34.29 0)
 			(effects
