File: SCRController/Design/SCRController/SCRController.kicad_pcb (KiCad board)
At the start: 2 copper layers, 77.6 x 73.5 mm, 43 parts, among them J1 VALT, J2 SAL_TRIAC, Q1 2N2907A, Q2 2N2222A, Q3 2N2222A, Q4 2N2907A, U1 TL084, U2 TL084, U3 LM7815_TO220, U4 LM7915_TO220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

Commit message: a
Parts:
- C2, C5: footprint Capacitor_THT:C_Radial_D4.0mm_H5.0mm_P1.50mm -> Capacitor_THT:C_Radial_D12.5mm_H25.0mm_P5.00mm
- Q1, Q2, Q3, Q4: footprint Package_TO_SOT_THT:TO-92L_Inline -> Package_TO_SOT_THT:TO-92L_Inline_Wide
- moved C5 44.5 mm to (71.9, 83.7)
- moved C2 33.1 mm to (98.8, 90.3), turned to 180 degrees
- moved Q4 4.18 mm to (69.8, 62.2), turned to 90 degrees
- moved R7 3.41 mm to (94.3, 73.6)
- moved D1 3.31 mm to (101.1, 81.0)
- moved Q3 2.47 mm to (58.4, 56.8)
- moved Q2 1.93 mm to (54.3, 29.9)
Connections:
- U1 pad 12: VCOMP -> Net-(Q2-C)
- U1 pad 13: Net-(Q2-C) -> VCOMP
Routing:
- net VDC-: track 75.2 -> 109.0 mm
- net Earth: track 452.9 -> 485.1 mm
- net VSync: track 176.6 -> 186.2 mm
- net Net-(Q4-C): track 32.0 -> 25.8 mm
- net Net-(Q4-E): track 9.35 -> 5.04 mm
- net Net-(Q3-B): track 5.88 -> 8.92 mm
- net VA-: track 10.8 -> 8.08 mm
- net VA+: track 22.4 -> 19.7 mm
- net A2: track 55.7 -> 57.9 mm
- net VDC+: track 38.1 -> 39.9 mm
- net VCC: track 190.9 -> 189.4 mm
- net Net-(Q2-B): track 9.00 -> 7.59 mm
- net Net-(Q1-C): track 9.54 -> 10.6 mm
- net Net-(Q1-B): track 29.3 -> 30.0 mm
- net Net-(Q4-B): track 12.3 -> 11.7 mm
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Other:
- board size 77.6 x 73.5 mm -> 77.6 x 78.1 mm
