File: SCRController/Design/SCRController/SCRController.kicad_sch (KiCad schematic)
At the start: 41 parts, among them J1 VALT, J2 SAL_TRIAC, Q1 2N2907A, Q2 2N2222A, Q3 2N2222A, Q4 2N2907A, U1 TL084, U2 TL084, U3 LM7815_TO220, U4 LM7915_TO220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

Commit message: Updated footprints
Parts:
- D1: footprint Diode_THT:Diode_Bridge_GeneSiC_KBPC_W -> PCM_Diode_THT_AKL:Diode_Bridge_KBP
- J1: footprint (none) -> TerminalBlock:TerminalBlock_MaiXu_MX126-5.0-03P_1x03_P5.00mm
- J2: footprint (none) -> TerminalBlock:TerminalBlock_MaiXu_MX126-5.0-02P_1x02_P5.00mm
- U5: footprint (none) -> PCM_Package_DIP_AKL:DIP-6_W7.62mm_LongPads
Other:
- moved on the sheet: J1
Changed lines of the file:
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@@
 	)
 	(junction
-		(at 268.224 144.018)
+		(at 263.652 100.076)
 		(diameter 0)
 		(color 0 0 0 0)
@@
 	(wire
 		(pts
-			(xy 266.954 144.018) (xy 266.954 144.272)
+			(xy 262.382 100.076) (xy 262.382 100.33)
 		)
 		(stroke
@@
 	(wire
 		(pts
-			(xy 269.748 144.018) (xy 268.224 144.018)
+			(xy 265.176 100.076) (xy 263.652 100.076)
 		)
 		(stroke
@@
 	(wire
 		(pts
-			(xy 270.002 141.732) (xy 266.954 141.732)
+			(xy 265.43 97.79) (xy 262.382 97.79)
 		)
 		(stroke
@@
 	(wire
 		(pts
-			(xy 268.224 144.018) (xy 266.954 144.018)
+			(xy 263.652 100.076) (xy 262.382 100.076)
 		)
 		(stroke
@@
 	(wire
 		(pts
-			(xy 270.002 139.446) (xy 270.002 141.732)
+			(xy 265.43 95.504) (xy 265.43 97.79)
 		)
 		(stroke
@@
 	(wire
 		(pts
-			(xy 266.954 148.59) (xy 266.954 146.812)
+			(xy 262.382 104.648) (xy 262.382 102.87)
 		)
 		(stroke
@@
 	(wire
 		(pts
-			(xy 270.51 148.59) (xy 266.954 148.59)
+			(xy 265.938 104.648) (xy 262.382 104.648)
 		)
 		(stroke
@@
 	(wire
 		(pts
-			(xy 270.002 139.446) (xy 270.256 139.446)
+			(xy 265.43 95.504) (xy 265.684 95.504)
 		)
 		(stroke
@@
 	(global_label "DERCENT"
 		(shape input)
-		(at 269.748 144.018 0)
+		(at 265.176 100.076 0)
 		(fields_autoplaced yes)
 		(effects
@@
 		)
 		(property "Intersheetrefs" "${INTERSHEET_REFS}"
-			(at 281.1393 144.018 0)
+			(at 276.5673 100.076 0)
 			(effects
 				(font
@@
 	(global_label "VA+"
 		(shape input)
-		(at 270.256 139.446 0)
+		(at 265.684 95.504 0)
 		(fields_autoplaced yes)
 		(effects
@@
 		)
 		(property "Intersheetrefs" "${INTERSHEET_REFS}"
-			(at 276.9908 139.446 0)
+			(at 272.4188 95.504 0)
 			(effects
 				(font
@@
 	(global_label "VA-"
 		(shape input)
-		(at 270.51 148.59 0)
+		(at 265.938 104.648 0)
 		(fields_autoplaced yes)
 		(effects
@@
 		)
 		(property "Intersheetrefs" "${INTERSHEET_REFS}"
-			(at 277.2448 148.59 0)
+			(at 272.6728 104.648 0)
 			(effects
 				(font
@@
 	(symbol
 		(lib_id "power:Earth")
-		(at 268.224 144.018 0)
+		(at 263.652 100.076 0)
 		(unit 1)
 		(exclude_from_sim no)
@@
 		(fields_autoplaced yes)
 		(property "Reference" "#PWR013"
-			(at 268.224 150.368 0)
+			(at 263.652 106.426 0)
 			(effects
 				(font
@@
 		)
 		(property "Value" "Earth"
-			(at 268.224 149.352 0)
+			(at 263.652 105.41 0)
 			(effects
 				(font
@@
 		)
 		(property "Footprint" ""
-			(at 268.224 144.018 0)
+			(at 263.652 100.076 0)
 			(effects
 				(font
@@
 		)
 		(property "Datasheet" "~"
-			(at 268.224 144.018 0)
+			(at 263.652 100.076 0)
 			(effects
 				(font
@@
 		)
 		(property "Description" "Power symbol creates a global label with name \"Earth\""
-			(at 268.224 144.018 0)
+			(at 263.652 100.076 0)
 			(effects
 				(font
@@
 	(symbol
 		(lib_id "Connector:Conn_01x03_Pin")
-		(at 261.874 144.272 0)
+		(at 257.302 100.33 0)
 		(unit 1)
 		(exclude_from_sim no)
@@
 		(fields_autoplaced yes)
 		(property "Reference" "J1"
-			(at 262.509 137.16 0)
+			(at 257.937 93.218 0)
 			(effects
 				(font
@@
 		)
 		(property "Value" "VALT"
-			(at 262.509 139.7 0)
+			(at 257.937 95.758 0)
 			(effects
 				(font
@@
 			)
 		)
-		(property "Footprint" ""
-			(at 261.874 144.272 0)
+		(property "Footprint" "TerminalBlock:TerminalBlock_MaiXu_MX126-5.0-03P_1x03_P5.00mm"
+			(at 257.302 100.33 0)
 			(effects
 				(font
@@
 		)
 		(property "Datasheet" "~"
-			(at 261.874 144.272 0)
+			(at 257.302 100.33 0)
 			(effects
 				(font
@@
 		)
 		(property "Description" "Generic connector, single row, 01x03, script generated"
-			(at 261.874 144.272 0)
+			(at 257.302 100.33 0)
 			(effects
 				(font
@@
 			)
 		)
-		(property "Footprint" "Diode_THT:Diode_Bridge_GeneSiC_KBPC_W"
+		(property "Footprint" "PCM_Diode_THT_AKL:Diode_Bridge_KBP"
 			(at 233.934 125.984 0)
 			(effects
@@
 			)
 		)
-		(property "Footprint" ""
+		(property "Footprint" "TerminalBlock:TerminalBlock_MaiXu_MX126-5.0-02P_1x02_P5.00mm"
 			(at 255.524 83.566 0)
 			(effects
@@
 			)
 		)
-		(property "Footprint" ""
+		(property "Footprint" "PCM_Package_DIP_AKL:DIP-6_W7.62mm_LongPads"
 			(at 218.694 89.916 0)
 			(effects

Commit message: Update SCRController design files
Parts:
- added RV1: R_Potentiometer_US, Potentiometer_THT:Potentiometer_Alps_RK09Y11_Single_Horizontal, symbol Device:R_Potentiometer_US
- D3, D4, D6: footprint Resistor_THT:R_Axial_DIN0207_L6.3mm_D2.5mm_P7.62mm_Horizontal -> PCM_Diode_THT_AKL:Diode_Bridge_KBP
Connections:
- net Earth: now also RV1.3
- net VCC: now also RV1.1
- net VCOMP: now also RV1.2
Changed lines of the file:
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@@
 	(wire
 		(pts
+			(xy 148.59 163.83) (xy 148.59 167.64)
+		)
+		(stroke
+			(width 0)
+			(type default)
+		)
+	)
+	(wire
+		(pts
 			(xy 97.79 57.15) (xy 105.41 57.15)
 		)
@@
 	(wire
 		(pts
+			(xy 148.59 175.26) (xy 148.59 180.34)
+		)
+		(stroke
+			(width 0)
+			(type default)
+		)
+	)
+	(wire
+		(pts
 			(xy 88.9 20.32) (xy 97.79 20.32)
 		)
@@
 		)
 	)
+	(global_label "VCC"
+		(shape input)
+		(at 148.59 163.83 0)
+		(fields_autoplaced yes)
+		(effects
+			(font
+				(size 1.27 1.27)
+			)
+			(justify left)
+		)
+		(property "Intersheetrefs" "${INTERSHEET_REFS}"
+			(at 155.2038 163.83 0)
+			(effects
+				(font
+					(size 1.27 1.27)
+				)
+				(justify left)
+				(hide yes)
+			)
+		)
+	)
 	(global_label "VEE"
 		(shape input)
@@
 		)
 	)
+	(global_label "VCOMP"
+		(shape input)
+		(at 152.4 171.45 0)
+		(fields_autoplaced yes)
+		(effects
+			(font
+				(size 1.27 1.27)
+			)
+			(justify left)
+		)
+		(property "Intersheetrefs" "${INTERSHEET_REFS}"
+			(at 161.7957 171.45 0)
+			(effects
+				(font
+					(size 1.27 1.27)
+				)
+				(justify left)
+				(hide yes)
+			)
+		)
+	)
 	(global_label "VCC"
 		(shape input)
@@
 			)
 		)
-		(property "Footprint" "Resistor_THT:R_Axial_DIN0207_L6.3mm_D2.5mm_P7.62mm_Horizontal"
+		(property "Footprint" "PCM_Diode_THT_AKL:Diode_Bridge_KBP"
 			(at 135.89 132.08 0)
 			(effects
@@
 	)
 	(symbol
+		(lib_id "Device:R_Potentiometer_US")
+		(at 148.59 171.45 0)
+		(unit 1)
+		(exclude_from_sim no)
+		(in_bom yes)
+		(on_board yes)
+		(dnp no)
+		(fields_autoplaced yes)
+		(property "Reference" "RV1"
+			(at 146.05 170.1799 0)
+			(effects
+				(font
+					(size 1.27 1.27)
+				)
+				(justify right)
+			)
+		)
+		(property "Value" "R_Potentiometer_US"
+			(at 146.05 172.7199 0)
+			(effects
+				(font
+					(size 1.27 1.27)
+				)
+				(justify right)
+			)
+		)
+		(property "Footprint" "Potentiometer_THT:Potentiometer_Alps_RK09Y11_Single_Horizontal"
+			(at 148.59 171.45 0)
+			(effects
+				(font
+					(size 1.27 1.27)
+				)
+				(hide yes)
+			)
+		)
+		(property "Datasheet" "~"
+			(at 148.59 171.45 0)
+			(effects
+				(font
+					(size 1.27 1.27)
+				)
+				(hide yes)
+			)
+		)
+		(property "Description" "Potentiometer, US symbol"
+			(at 148.59 171.45 0)
+			(effects
+				(font
+					(size 1.27 1.27)
+				)
+				(hide yes)
+			)
+		)
+		(pin "3"
+		)
+		(pin "1"
+		)
+		(pin "2"
+		)
+		(instances
+			(project ""
+				(path "/3415e815-e6d7-4ea4-b663-6aaf90e60fb1"
+					(reference "RV1")
+					(unit 1)
+				)
+			)
+		)
+	)
+	(symbol
+		(lib_id "power:Earth")
+		(at 148.59 180.34 0)
+		(unit 1)
+		(exclude_from_sim no)
+		(in_bom yes)
+		(on_board yes)
+		(dnp no)
+		(fields_autoplaced yes)
+		(property "Reference" "#PWR014"
+			(at 148.59 186.69 0)
+			(effects
+				(font
+					(size 1.27 1.27)
+				)
+				(hide yes)
+			)
+		)
+		(property "Value" "Earth"
+			(at 148.59 185.42 0)
+			(effects
+				(font
+					(size 1.27 1.27)
+				)
+				(hide yes)
+			)
+		)
+		(property "Footprint" ""
+			(at 148.59 180.34 0)
+			(effects
+				(font
+					(size 1.27 1.27)
+				)
+				(hide yes)
+			)
+		)
+		(property "Datasheet" "~"
+			(at 148.59 180.34 0)
+			(effects
+				(font
+					(size 1.27 1.27)
+				)
+				(hide yes)
+			)
+		)
+		(property "Description" "Power symbol creates a global label with name \"Earth\""
+			(at 148.59 180.34 0)
+			(effects
+				(font
+					(size 1.27 1.27)
+				)
+				(hide yes)
+			)
+		)
+		(pin "1"
+		)
+		(instances
+			(project "SCRController"
+				(path "/3415e815-e6d7-4ea4-b663-6aaf90e60fb1"
+					(reference "#PWR014")
+					(unit 1)
+				)
+			)
+		)
+	)
+	(symbol
 		(lib_id "PCM_Capacitor_AKL:C_Disc_D3.0mm_W1.6mm_P2.50mm")
 		(at 90.17 123.19 0)
@@
 			)
 		)
-		(property "Footprint" "Resistor_THT:R_Axial_DIN0207_L6.3mm_D2.5mm_P7.62mm_Horizontal"
+		(property "Footprint" "PCM_Diode_THT_AKL:Diode_Bridge_KBP"
 			(at 135.89 64.77 0)
 			(effects
@@
 			)
 		)
-		(property "Footprint" "Resistor_THT:R_Axial_DIN0207_L6.3mm_D2.5mm_P7.62mm_Horizontal"
+		(property "Footprint" "PCM_Diode_THT_AKL:Diode_Bridge_KBP"
 			(at 58.42 68.58 0)
 			(effects

Commit message: Changed FP
Parts:
- D3, D4, D6: footprint PCM_Diode_THT_AKL:Diode_Bridge_KBP -> Diode_THT:D_DO-15_P5.08mm_Vertical_AnodeUp
Changed lines of the file:
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@@
 			)
 		)
-		(property "Footprint" "PCM_Diode_THT_AKL:Diode_Bridge_KBP"
+		(property "Footprint" "Diode_THT:D_DO-15_P5.08mm_Vertical_AnodeUp"
 			(at 135.89 132.08 0)
 			(effects
@@
 			)
 		)
-		(property "Footprint" "PCM_Diode_THT_AKL:Diode_Bridge_KBP"
+		(property "Footprint" "Diode_THT:D_DO-15_P5.08mm_Vertical_AnodeUp"
 			(at 135.89 64.77 0)
 			(effects
@@
 			)
 		)
-		(property "Footprint" "PCM_Diode_THT_AKL:Diode_Bridge_KBP"
+		(property "Footprint" "Diode_THT:D_DO-15_P5.08mm_Vertical_AnodeUp"
 			(at 58.42 68.58 0)
 			(effects

Commit message: Pcb full
Parts:
- C2, C5: value C -> 2200uF
- C4, C6: value C -> 0.1uF
- RV1: value R_Potentiometer_US -> 5K
Connections:
- net Earth: now also U4.1 (GND)
Changed lines of the file:
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@@
 	(wire
 		(pts
+			(xy 225.044 164.084) (xy 225.298 164.084)
+		)
+		(stroke
+			(width 0)
+			(type default)
+		)
+	)
+	(wire
+		(pts
 			(xy 144.78 132.08) (xy 144.78 135.89)
 		)
@@
 			)
 		)
-		(property "Value" "C"
+		(property "Value" "0.1uF"
 			(at 244.094 149.0979 0)
 			(effects
@@
 			)
 		)
-		(property "Value" "R_Potentiometer_US"
+		(property "Value" "5K"
 			(at 146.05 172.7199 0)
 			(effects
@@
 		(fields_autoplaced yes)
 		(property "Reference" "C6"
-			(at 238.506 164.8459 0)
+			(at 237.49 164.8459 0)
 			(effects
 				(font
@@
 			)
 		)
-		(property "Value" "C"
-			(at 238.506 167.3859 0)
+		(property "Value" "0.1uF"
+			(at 237.49 167.3859 0)
 			(effects
 				(font
@@
 		(fields_autoplaced yes)
 		(property "Reference" "C5"
-			(at 221.488 162.5599 0)
+			(at 219.71 162.5599 0)
 			(effects
 				(font
@@
 			)
 		)
-		(property "Value" "C"
-			(at 221.488 165.0999 0)
+		(property "Value" "2200uF"
+			(at 219.71 165.0999 0)
 			(effects
 				(font
@@
 		(fields_autoplaced yes)
 		(property "Reference" "C2"
-			(at 221.996 144.2719 0)
+			(at 220.98 144.2719 0)
 			(effects
 				(font
@@
 			)
 		)
-		(property "Value" "C"
-			(at 221.996 146.8119 0)
+		(property "Value" "2200uF"
+			(at 220.98 146.8119 0)
 			(effects
 				(font

Commit message: Correcciones
Parts:
- added R20: 10k, Resistor_THT:R_Axial_DIN0207_L6.3mm_D2.5mm_P7.62mm_Horizontal, symbol Device:R
- RV1: footprint Potentiometer_THT:Potentiometer_Alps_RK09Y11_Single_Horizontal -> Potentiometer_THT:Potentiometer_Alps_RK163_Single_Horizontal
Connections:
- net SUM: now also R20.1; no longer U5.1
- net VA+: now also D1.3 (-); no longer D1.4
- net VDC-: now also D1.4; no longer D1.3 (-)
- new net: R20.2, U5.1
Changed lines of the file:
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@@
 	)
 	(junction
-		(at 263.652 100.076)
-		(diameter 0)
-		(color 0 0 0 0)
-	)
-	(junction
 		(at 183.896 105.41)
 		(diameter 0)
@@
 	(wire
 		(pts
+			(xy 244.856 110.744) (xy 241.554 110.744)
+		)
+		(stroke
+			(width 0)
+			(type default)
+		)
+	)
+	(wire
+		(pts
 			(xy 80.01 62.23) (xy 116.84 62.23)
 		)
@@
 	(wire
 		(pts
-			(xy 265.176 100.076) (xy 263.652 100.076)
-		)
-		(stroke
-			(width 0)
-			(type default)
-		)
-	)
-	(wire
-		(pts
 			(xy 265.43 97.79) (xy 262.382 97.79)
 		)
@@
 	(wire
 		(pts
-			(xy 97.79 16.51) (xy 97.79 20.32)
+			(xy 196.85 82.042) (xy 208.28 82.042)
 		)
 		(stroke
@@
 	(wire
 		(pts
-			(xy 36.83 101.6) (xy 36.83 137.16)
+			(xy 97.79 16.51) (xy 97.79 20.32)
 		)
 		(stroke
@@
 	(wire
 		(pts
-			(xy 80.01 50.8) (xy 80.01 43.18)
+			(xy 36.83 101.6) (xy 36.83 137.16)
 		)
 		(stroke
@@
 	(wire
 		(pts
-			(xy 241.554 110.998) (xy 241.554 110.744)
+			(xy 80.01 50.8) (xy 80.01 43.18)
 		)
 		(stroke
@@
 	(wire
 		(pts
-			(xy 216.154 82.55) (xy 216.154 82.296)
+			(xy 216.154 82.042) (xy 216.154 82.296)
 		)
 		(stroke
@@
 	(wire
 		(pts
-			(xy 223.266 110.744) (xy 226.314 110.744)
-		)
-		(stroke
-			(width 0)
-			(type default)
-		)
-	)
-	(wire
-		(pts
 			(xy 88.9 57.15) (xy 88.9 55.88)
 		)
@@
 	(wire
 		(pts
-			(xy 233.934 96.266) (xy 234.188 96.266)
-		)
-		(stroke
-			(width 0)
-			(type default)
-		)
-	)
-	(wire
-		(pts
 			(xy 90.17 95.25) (xy 90.17 91.44)
 		)
@@
 	(wire
 		(pts
-			(xy 243.078 110.998) (xy 241.554 110.998)
-		)
-		(stroke
-			(width 0)
-			(type default)
-		)
-	)
-	(wire
-		(pts
 			(xy 217.424 171.704) (xy 216.408 171.704)
 		)
@@
 	(wire
 		(pts
-			(xy 212.344 82.55) (xy 216.154 82.55)
-		)
-		(stroke
-			(width 0)
-			(type default)
-		)
-	)
-	(wire
-		(pts
 			(xy 55.88 139.7) (xy 52.07 139.7)
 		)
@@
 	(wire
 		(pts
+			(xy 226.314 110.744) (xy 222.504 110.744)
+		)
+		(stroke
+			(width 0)
+			(type default)
+		)
+	)
+	(wire
+		(pts
 			(xy 105.41 36.83) (xy 105.41 45.72)
 		)
@@
 	(wire
 		(pts
-			(xy 223.266 117.094) (xy 223.266 110.744)
+			(xy 227.584 103.124) (xy 233.934 103.124)
 		)
 		(stroke
@@
 	(wire
 		(pts
-			(xy 233.934 103.124) (xy 233.934 96.266)
+			(xy 80.01 43.18) (xy 88.9 43.18)
 		)
 		(stroke
@@
 	(wire
 		(pts
-			(xy 80.01 43.18) (xy 88.9 43.18)
+			(xy 241.046 141.986) (xy 239.014 141.986)
 		)
 		(stroke
@@
 	(wire
 		(pts
-			(xy 241.046 141.986) (xy 239.014 141.986)
+			(xy 144.78 132.08) (xy 146.05 132.08)
 		)
 		(stroke
@@
 	(wire
 		(pts
-			(xy 144.78 132.08) (xy 146.05 132.08)
+			(xy 88.9 24.13) (xy 88.9 20.32)
 		)
 		(stroke
@@
 	(wire
 		(pts
-			(xy 88.9 24.13) (xy 88.9 20.32)
+			(xy 81.28 129.54) (xy 81.28 134.62)
 		)
 		(stroke
@@
 	(wire
 		(pts
-			(xy 81.28 129.54) (xy 81.28 134.62)
+			(xy 259.334 161.544) (xy 258.826 161.544)
 		)
 		(stroke
@@
 	(wire
 		(pts
-			(xy 259.334 161.544) (xy 258.826 161.544)
+			(xy 114.3 67.31) (xy 116.84 67.31)
 		)
 		(stroke
@@
 	(wire
 		(pts
-			(xy 114.3 67.31) (xy 116.84 67.31)
+			(xy 222.504 110.744) (xy 222.504 114.3)
 		)
 		(stroke
@@
 	(wire
 		(pts
+			(xy 215.9 82.042) (xy 216.154 82.042)
+		)
+		(stroke
+			(width 0)
+			(type default)
+		)
+	)
+	(wire
+		(pts
 			(xy 232.664 171.704) (xy 233.426 171.704)
 		)
@@
 	(global_label "VA+"
 		(shape input)
-		(at 234.188 96.266 0)
-		(fields_autoplaced yes)
-		(effects
-			(font
-				(size 1.27 1.27)
-			)
-			(justify left)
-		)
-		(property "Intersheetrefs" "${INTERSHEET_REFS}"
-			(at 240.9228 96.266 0)
-			(effects
-				(font
-					(size 1.27 1.27)
-				)
-				(justify left)
-				(hide yes)
-			)
-		)
-	)
-	(global_label "DERCENT"
-		(shape input)
-		(at 265.176 100.076 0)
+		(at 222.504 114.3 180)
 		(fields_autoplaced yes)
 		(effects
@@
 				(size 1.27 1.27)
 			)
-			(justify left)
+			(justify right)
 		)
 		(property "Intersheetrefs" "${INTERSHEET_REFS}"
-			(at 276.5673 100.076 0)
+			(at 215.7692 114.3 0)
 			(effects
 				(font
 					(size 1.27 1.27)
 				)
-				(justify left)
+				(justify right)
 				(hide yes)
 			)
@@
 	(global_label "VDC-"
 		(shape input)
-		(at 223.266 117.094 270)
+		(at 227.584 103.124 180)
 		(fields_autoplaced yes)
 		(effects
@@
 		)
 		(property "Intersheetrefs" "${INTERSHEET_REFS}"
-			(at 223.266 125.2802 90)
+			(at 219.3978 103.124 0)
 			(effects
 				(font
@@
 	(global_label "VDC+"
 		(shape input)
-		(at 243.078 110.998 0)
+		(at 244.856 110.744 0)
 		(fields_autoplaced yes)
 		(effects
@@
 		)
 		(property "Intersheetrefs" "${INTERSHEET_REFS}"
-			(at 251.2642 110.998 0)
+			(at 253.0422 110.744 0)
 			(effects
 				(font
@@
 	(global_label "SUM"
 		(shape input)
-		(at 212.344 82.55 180)
+		(at 196.85 82.042 180)
 		(fields_autoplaced yes)
 		(effects
@@
 		)
 		(property "Intersheetrefs" "${INTERSHEET_REFS}"
-			(at 205.3674 82.55 0)
+			(at 189.8734 82.042 0)
 			(effects
 				(font
@@
 			)
 		)
-		(property "Footprint" "Potentiometer_THT:Potentiometer_Alps_RK09Y11_Single_Horizontal"
+		(property "Footprint" "Potentiometer_THT:Potentiometer_Alps_RK163_Single_Horizontal"
 			(at 148.59 171.45 0)
 			(effects
@@
 					(unit 1)
 				)
+			)
+		)
+	)
+	(symbol
+		(lib_id "Device:R")
+		(at 212.09 82.042 90)
+		(unit 1)
+		(exclude_from_sim no)
+		(in_bom yes)
+		(on_board yes)
+		(dnp no)
+		(fields_autoplaced yes)
+		(property "Reference" "R20"
+			(at 212.09 75.946 90)
+			(effects
+				(font
+					(size 1.27 1.27)
+				)
+			)
+		)
+		(property "Value" "10k"
+			(at 212.09 78.486 90)
+			(effects
+				(font
+					(size 1.27 1.27)
+				)
+			)
+		)
+		(property "Footprint" "Resistor_THT:R_Axial_DIN0207_L6.3mm_D2.5mm_P7.62mm_Horizontal"
+			(at 212.09 83.82 90)
+			(effects
+				(font
+					(size 1.27 1.27)
+				)
+				(hide yes)
+			)
+		)
+		(property "Datasheet" "~"
+			(at 212.09 82.042 0)
+			(effects
+				(font
+					(size 1.27 1.27)
+				)
+				(hide yes)
+			)
+		)
+		(property "Description" "Resistor"
+			(at 212.09 82.042 0)
+			(effects
+				(font
+					(size 1.27 1.27)
+				)
+				(hide yes)
+			)
+		)
+		(pin "2"
+		)
+		(pin "1"
+		)
+		(instances
+			(project "SCRController"
+				(path "/3415e815-e6d7-4ea4-b663-6aaf90e60fb1"
+					(reference "R20")
+					(unit 1)
+				)

Commit message: a
Parts:
- C2, C5: footprint Capacitor_THT:C_Radial_D4.0mm_H5.0mm_P1.50mm -> Capacitor_THT:C_Radial_D12.5mm_H25.0mm_P5.00mm
- Q1, Q2, Q3, Q4: footprint Package_TO_SOT_THT:TO-92L_Inline -> Package_TO_SOT_THT:TO-92L_Inline_Wide
Connections:
- net VCOMP: now also U1.13 (-); no longer U1.12 (+)
- net at Q2.3 (C), R15.2: now also U1.12 (+); no longer U1.13 (-)
Changed lines of the file:
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@@
 	)
 	(junction
-		(at 81.28 134.62)
-		(diameter 0)
-		(color 0 0 0 0)
-	)
-	(junction
 		(at 239.014 141.986)
 		(diameter 0)
@@
 		(color 0 0 0 0)
 	)
+	(junction
+		(at 81.28 133.096)
+		(diameter 0)
+		(color 0 0 0 0)
+	)
 	(wire
 		(pts
@@
 	(wire
 		(pts
-			(xy 170.18 114.554) (xy 166.116 114.554)
+			(xy 116.84 129.54) (xy 116.84 133.096)
 		)
 		(stroke
@@
 	(wire
 		(pts
-			(xy 216.408 156.21) (xy 222.758 156.21)
+			(xy 170.18 114.554) (xy 166.116 114.554)
 		)
 		(stroke
@@
 	(wire
 		(pts
-			(xy 262.382 100.076) (xy 262.382 100.33)
+			(xy 216.408 156.21) (xy 222.758 156.21)
 		)
 		(stroke
@@
 	(wire
 		(pts
-			(xy 211.836 171.704) (xy 216.408 171.704)
+			(xy 262.382 100.076) (xy 262.382 100.33)
 		)
 		(stroke
@@
 	(wire
 		(pts
-			(xy 29.718 20.574) (xy 29.718 21.59)
+			(xy 211.836 171.704) (xy 216.408 171.704)
 		)
 		(stroke
@@
 	(wire
 		(pts
-			(xy 244.856 110.744) (xy 241.554 110.744)
+			(xy 29.718 20.574) (xy 29.718 21.59)
 		)
 		(stroke
@@
 	(wire
 		(pts
-			(xy 80.01 62.23) (xy 116.84 62.23)
+			(xy 244.856 110.744) (xy 241.554 110.744)
 		)
 		(stroke
@@
 	(wire
 		(pts
-			(xy 81.28 134.62) (xy 116.84 134.62)
+			(xy 80.01 62.23) (xy 116.84 62.23)
 		)
 		(stroke
@@
 	(wire
 		(pts
-			(xy 114.3 129.54) (xy 116.84 129.54)
+			(xy 90.17 91.44) (xy 99.06 91.44)
 		)
 		(stroke
@@
 	(wire
 		(pts
-			(xy 90.17 91.44) (xy 99.06 91.44)
+			(xy 239.014 156.464) (xy 233.426 156.464)
 		)
 		(stroke
@@
 	(wire
 		(pts
-			(xy 239.014 156.464) (xy 233.426 156.464)
+			(xy 97.79 107.95) (xy 106.68 107.95)
 		)
 		(stroke
@@
 	(wire
 		(pts
-			(xy 97.79 107.95) (xy 106.68 107.95)
+			(xy 236.22 81.28) (xy 231.394 81.28)
 		)
 		(stroke
@@
 	(wire
 		(pts
-			(xy 236.22 81.28) (xy 231.394 81.28)
+			(xy 81.28 133.096) (xy 81.28 134.62)
 		)
 		(stroke
@@
 	(wire
 		(pts
+			(xy 81.28 133.096) (xy 116.84 133.096)
+		)
+		(stroke
+			(width 0)
+			(type default)
+		)
+	)
+	(wire
+		(pts
 			(xy 193.802 105.41) (xy 183.896 105.41)
 		)
@@
 	(wire
 		(pts
-			(xy 114.3 129.54) (xy 114.3 96.52)
+			(xy 114.3 96.52) (xy 114.3 134.62)
 		)
 		(stroke
@@
 	(wire
 		(pts
+			(xy 114.3 134.62) (xy 116.84 134.62)
+		)
+		(stroke
+			(width 0)
+			(type default)
+		)
+	)
+	(wire
+		(pts
 			(xy 216.916 149.352) (xy 216.408 149.352)
 		)
@@
 	(wire
 		(pts
-			(xy 81.28 129.54) (xy 81.28 134.62)
+			(xy 81.28 129.54) (xy 81.28 133.096)
 		)
 		(stroke
@@
 			)
 		)
-		(property "Footprint" "Package_TO_SOT_THT:TO-92L_Inline"
+		(property "Footprint" "Package_TO_SOT_THT:TO-92L_Inline_Wide"
 			(at 82.55 66.04 0)
 			(effects
@@
 			)
 		)
-		(property "Footprint" "Package_TO_SOT_THT:TO-92L_Inline"
+		(property "Footprint" "Package_TO_SOT_THT:TO-92L_Inline_Wide"
 			(at 83.82 137.16 0)
 			(effects
@@
 			)
 		)
-		(property "Footprint" "Capacitor_THT:C_Radial_D4.0mm_H5.0mm_P1.50mm"
+		(property "Footprint" "Capacitor_THT:C_Radial_D12.5mm_H25.0mm_P5.00mm"
 			(at 217.3732 167.64 0)
 			(effects
@@
 			)
 		)
-		(property "Footprint" "Capacitor_THT:C_Radial_D4.0mm_H5.0mm_P1.50mm"
+		(property "Footprint" "Capacitor_THT:C_Radial_D12.5mm_H25.0mm_P5.00mm"
 			(at 217.8812 149.352 0)
 			(effects
@@
 			)
 		)
-		(property "Footprint" "Package_TO_SOT_THT:TO-92L_Inline"
+		(property "Footprint" "Package_TO_SOT_THT:TO-92L_Inline_Wide"
 			(at 87.63 105.41 0)
 			(effects
@@
 			)
 		)
-		(property "Footprint" "Package_TO_SOT_THT:TO-92L_Inline"
+		(property "Footprint" "Package_TO_SOT_THT:TO-92L_Inline_Wide"
 			(at 86.36 34.29 0)
 			(effects
